File: fourier/fourier.sch (KiCad schematic (older format))
At the start: 94 parts, among them J1 VCC, J2 ICSP, J3 RGB1, J4 F4, J5 F5, J6 C6, J7 GND, Q1 MMBT3904, U1 TRRS, U6 TRRS, U7 ProMicro

Commit message: Fourier 1.0
Parts:
- removed D_D4, D_D6, D_E5, D_E6: D, Keebio-Parts:Diode-dual, symbol D
- removed J2: ICSP, Socket_Strips:Socket_Strip_Straight_1x06_Pitch2.54mm, symbol CONN_02X03
- removed J4: F4, Keebio-Parts:SinglePad, symbol TEST_1P
- removed J5: F5, Keebio-Parts:SinglePad, symbol TEST_1P
- removed Q1: MMBT3904, TO_SOT_Packages_SMD:SOT-23, symbol MMBT3904
- removed R3: 1k, Keebio-Parts:Resistor-Compact, symbol R
- removed R_A1, R_A2, R_A3, R_A4, R_A5, R_A6, R_B1, R_B2, R_B3, R_B4, R_B5, R_B6, R_C1, R_C2, R_C3, R_C4, R_C5, R_C6, R_D1, R_D2, R_D3, R_D4, R_D5, R_D6, R_E5, R_E6: R, Keebio-Parts:Resistor-Hybrid, symbol R
- removed SW_A1, SW_A2, SW_A3, SW_A4, SW_A5, SW_A6, SW_B1, SW_B2, SW_B3, SW_B4, SW_B5, SW_B6, SW_C1, SW_C2, SW_C3, SW_C4, SW_C5, SW_C6, SW_D1, SW_D2, SW_D3, SW_D4, SW_D5, SW_D6, SW_E5, SW_E6: MX, Keebio-Parts:Hybrid_PCB_100H_Dual_hole-LED, symbol MX
- removed U6: TRRS, Keebio-Parts:TRRS-PJ-320A, symbol TRRS
- added SW_A1, SW_A2, SW_A3, SW_A4, SW_A5, SW_A6, SW_B2, SW_B3, SW_B4, SW_B5, SW_B6, SW_C2, SW_C3, SW_C4, SW_C5, SW_C6, SW_D2: SW_PUSH, MX_Alps_Hybrid:MX-1U-NoLED, symbol SW_PUSH
- added SW_B1, SW_D1, SW_D3, SW_Db3: SW_PUSH, MX_Alps_Hybrid:MX-1.25U-NoLED, symbol SW_PUSH
- added SW_C1: SW_PUSH, MX_Alps_Hybrid:MX-1.75U-NoLED, symbol SW_PUSH
- added SW_D5: SW_PUSH, MX_Alps_Hybrid:MX-2.75U-NoLED, symbol SW_PUSH
- added SW_Db1, SW_Db2, SW_Dc3: SW_PUSH, MX_Alps_Hybrid:MX-1.5U-NoLED, symbol SW_PUSH
- added SW_Db5: SW_PUSH, MX_Alps_Hybrid:MX-2.25U-NoLED, symbol SW_PUSH
- J1, J3, J6, J7, W2: footprint Keebio-Parts:SinglePad -> Keebio-Parts:Single-Pad
- R1, R2: footprint Keebio-Parts:Resistor-Compact -> Keebio-Parts:Resistor-Hybrid
- U1: renamed from U7; footprint Keebio-Parts:ARDUINO_PRO_MICRO -> Keebio-Parts:ArduinoProMicro
- renumbered U1 to T1
Connections:
- net F4 is gone; now on net rowA: U1.20 (A3/PF4)
- net F5 is gone; now on net col1: U1.19 (A2/PF5)
- net col1: now also SW_A1.1, SW_B1.1, SW_C1.1, SW_D1.1, SW_Db1.1; no longer U1.18 (A1/PF6)
- net col2: now also U1.18 (A1/PF6), SW_A2.1, SW_B2.1, SW_C2.1, SW_D2.1, SW_Db2.2; no longer U1.17 (A0/PF7)
- net col3: now also U1.17 (A0/PF7), SW_A3.1, SW_B3.1, SW_C3.1, SW_D3.2, SW_Db3.1, SW_Dc3.1; no longer U1.16 (15/PB1)
- net col4: now also U1.16 (15/PB1), SW_A4.1, SW_B4.1, SW_C4.1; no longer U1.15 (14/PB3)
- net col5: now also U1.15 (14/PB3), SW_A5.1, SW_B5.1, SW_C5.1, SW_D5.2, SW_Db5.1; no longer U1.14 (16/PB2)
- net col6: now also U1.14 (16/PB2), SW_A6.1, SW_B6.1, SW_C6.1; no longer U1.13 (10/PB6)
- net rowA: no longer U1.9 (6/PD7)
- net rowB: now also U1.9 (6/PD7); no longer U1.10 (7/PE6)
- net rowC: now also U1.10 (7/PE6); no longer U1.11 (8/PB4)
- net rowD: now also U1.11 (8/PB4); no longer U1.2 (RX1/PD2)
- net at D_A1.2 (A): now also SW_A1.2
- net at D_B1.2 (A): now also SW_B1.2
- net at D_C1.2 (A): now also SW_C1.2
- net at D_D1.2 (A): now also SW_D1.2, SW_Db1.2
- net at D_A2.2 (A): now also SW_A2.2
- net at D_B2.2 (A): now also SW_B2.2
- net at D_C2.2 (A): now also SW_C2.2
- net at D_D2.2 (A): now also SW_D2.2, SW_Db2.1
- net at D_A3.2 (A): now also SW_A3.2
- net at D_B3.2 (A): now also SW_B3.2
- net at D_C3.2 (A): now also SW_C3.2
- net at D_D3.2 (A): now also SW_D3.1, SW_Db3.2, SW_Dc3.2
- net at D_A4.2 (A): now also SW_A4.2
- net at D_B4.2 (A): now also SW_B4.2
- net at D_C4.2 (A): now also SW_C4.2
- net at D_A5.2 (A): now also SW_A5.2
- net at D_B5.2 (A): now also SW_B5.2
- net at D_C5.2 (A): now also SW_C5.2
- net at D_D5.2 (A): now also SW_D5.1, SW_Db5.2
- net at D_A6.2 (A): now also SW_A6.2
- net at D_B6.2 (A): now also SW_B6.2
- net at D_C6.2 (A): now also SW_C6.2
- net rowE: no longer names the net of U1.7 (4/PD4)
Other:
- moved on the sheet: J1, J3, J6, J7, T1
