File: fourier/fourier-right/fourier-right-top.kicad_pcb (KiCad board)
At the start: 2 copper layers, 141.4 x 92.2 mm, 7 parts

Commit message: Added 1u support on bottom-left, stepped 1.25u support on right half
Other:
- outline, holes or cut-outs redrawn
Changed lines of the file:
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@@
-(kicad_pcb (version 4) (host pcbnew 4.0.7)
+(kicad_pcb (version 20171130) (host pcbnew "(5.0.0-rc2-dev-90-gfabbc48)")
   (general
-    (links 0)
-    (no_connects 0)
-    (area 13.992857 21.925 166.482143 114.575)
     (thickness 1.6)
     (drawings 808)
@@
     (visible_elements 7FFFFF7F)
     (pcbplotparams
-      (layerselection 0x010c0_80000001)
+      (layerselection 0x010c0_ffffffff)
       (usegerberextensions true)
+      (usegerberattributes false)
+      (usegerberadvancedattributes false)
+      (creategerberjobfile false)
       (excludeedgelayer true)
       (linewidth 0.100000)
@@
       (hpglpenspeed 20)
       (hpglpendiameter 15)
-      (hpglpenoverlay 2)
       (psnegative false)
       (psa4output false)
@@
   (gr_line (start 117.336075 103.183334) (end 116.536071 103.183334) (layer Edge.Cuts) (width 0.1))
   (gr_line (start 117.336075 103.783334) (end 117.336075 103.183334) (layer Edge.Cuts) (width 0.1))
-  (gr_line (start 143.242066 84.733334) (end 129.242065 84.733334) (layer Edge.Cuts) (width 0.1))
+  (gr_line (start 143.242066 84.733334) (end 124.479565 84.733334) (layer Edge.Cuts) (width 0.1))
   (gr_line (start 143.242066 84.133333) (end 143.242066 84.733334) (layer Edge.Cuts) (width 0.1))
   (gr_line (start 144.042069 84.133333) (end 143.242066 84.133333) (layer Edge.Cuts) (width 0.1))
@@
   (gr_line (start 143.242066 71.333332) (end 144.042069 71.333332) (layer Edge.Cuts) (width 0.1))
   (gr_line (start 143.242066 70.733333) (end 143.242066 71.333332) (layer Edge.Cuts) (width 0.1))
-  (gr_line (start 129.242065 70.733333) (end 143.242066 70.733333) (layer Edge.Cuts) (width 0.1))
-  (gr_line (start 129.242065 71.333332) (end 129.242065 70.733333) (layer Edge.Cuts) (width 0.1))
-  (gr_line (start 128.442078 71.333332) (end 129.242065 71.333332) (layer Edge.Cuts) (width 0.1))
-  (gr_line (start 128.442078 84.133333) (end 128.442078 71.333332) (layer Edge.Cuts) (width 0.1))
-  (gr_line (start 129.242065 84.133333) (end 128.442078 84.133333) (layer Edge.Cuts) (width 0.1))
-  (gr_line (start 129.242065 84.733334) (end 129.242065 84.133333) (layer Edge.Cuts) (width 0.1))
+  (gr_line (start 124.479565 70.733333) (end 143.242066 70.733333) (layer Edge.Cuts) (width 0.1))
+  (gr_line (start 124.479565 71.333332) (end 124.479565 70.733333) (layer Edge.Cuts) (width 0.1))
+  (gr_line (start 123.679578 71.333332) (end 124.479565 71.333332) (layer Edge.Cuts) (width 0.1))
+  (gr_line (start 123.679578 84.133333) (end 123.679578 71.333332) (layer Edge.Cuts) (width 0.1))
+  (gr_line (start 124.479565 84.133333) (end 123.679578 84.133333) (layer Edge.Cuts) (width 0.1))
+  (gr_line (start 124.479565 84.733334) (end 124.479565 84.133333) (layer Edge.Cuts) (width 0.1))
   (gr_line (start 117.048065 84.733334) (end 103.048065 84.733334) (layer Edge.Cuts) (width 0.1))
   (gr_line (start 117.048065 84.133333) (end 117.048065 84.733334) (layer Edge.Cuts) (width 0.1))
